Commit message: Update URDF for Puzzlebot: refine link properties Co-authored-by: EmanuelVegaGlz <emanuelvegaglz@users.noreply.github.com> Co-authored-by: Diego Quezada <diegoquezadaco@users.noreply.github.com> Co-authored-by: BrisaReyCa <brisa.reyes.castro@outlook.com>

File: puzzlebobt_description/urdf/puzzlebot.urdf (robot description, URDF)
Before this commit: robot puzzlebot, 5 links, 4 joints
Links:
- removed link caster_wheel
- removed link wheel_left
- removed link wheel_right
- added link caster_link, mass 0.05; collision sphere radius=0.015; visual mesh filename=package://puzzlebot_sim/meshes/Puzzlebot_Caster_Wheel.stl scale=1 1 1
- added link wheel_l_link, mass 0.2; collision cylinder length=0.02 radius=0.0325; visual mesh filename=package://puzzlebot_sim/meshes/Puzzlebot_Wheel.stl scale=1 1 1
- added link wheel_r_link, mass 0.2; collision cylinder length=0.02 radius=0.0325; visual mesh filename=package://puzzlebot_sim/meshes/Puzzlebot_Wheel.stl scale=1 1 1
- link base_link: mass None -> 2.0; geometry collision box size=0.20 0.19 0.06; visual mesh filename=package://puzzlebot_sim/meshes/Puzzlebot_Jetson_Lidar_Editi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 scale=1 1 1
Joints:
- removed joint caster_wheel_joint
- removed joint wheel_left_joint
- removed joint wheel_right_joint
- added joint caster_joint: type fixed, parent base_link, child caster_link, origin xyz=-0.095 0.0 -0.03 rpy=0 0 0
- added joint wheel_l_joint: type continuous, parent base_link, child wheel_l_link, origin xyz=0.052 0.095 -0.0025 rpy=0 0 0, axis 0 1 0
- added joint wheel_r_joint: type continuous, parent base_link, child wheel_r_link, origin xyz=0.052 -0.095 -0.0025 rpy=0 0 0, axis 0 1 0
- joint base_link_joint: origin xyz=0 0 0.05 rpy=0 0 0 -> xyz=0.0 0.0 0.05 rpy=0 0 0
