Commit message: Co-authored-by: Aldrick T <taldrick@gmail.com> Co-authored-by: Diego Quezada <diegoquezadaco@users.noreply.github.com> Co-authored-by: BrisaReyCa <brisa.reyes.castro@outlook.com>

File: puzzlebot_description/urdf/puzzlebot.urdf (robot description, URDF)
Before this commit: robot Puzzlebot_Jetson_Lidar_Ed., 5 links, 4 joints
Links:
- added link laser_link, mass 0.1; collision cylinder length=0.05 radius=0.02; visual cylinder length=0.05 radius=0.02
- link base_link: geometry collision box size=0.20 0.19 0.06; visual mesh filename=package://puzzlebot_description/meshes/Puzzlebot_Jetson_Lid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 scale=1 1 1
- link caster_link: geometry collision sphere radius=0.015; visual sphere radius=0.015
- link wheel_l_link: geometry collision cylinder length=0.02 radius=0.0325; visual mesh filename=package://puzzlebot_description/meshes/Puzzlebot_Wheel.stl
- link wheel_r_link: geometry collision cylinder length=0.02 radius=0.0325; visual mesh filename=package://puzzlebot_description/meshes/Puzzlebot_Wheel.stl
Joints:
- added joint laser_joint: type fixed, parent base_link, child laser_link, origin xyz=0.08 0 0.10
- joint base_link_joint: origin xyz=0.0 0.0 0.05 rpy=0 0 0 -> xyz=0 0 0.05
- joint caster_joint: origin xyz=-0.095 0.0 -0.03 rpy=0 0 0 -> xyz=-0.09 0.0 -0.03
- joint wheel_l_joint: origin xyz=0.052 0.095 -0.0025 rpy=0 0 0 -> xyz=0.05 0.095 -0.02
- joint wheel_r_joint: origin xyz=0.052 -0.095 -0.0025 rpy=0 0 0 -> xyz=0.05 -0.095 -0.02

Commit message: feat: Update SLAM configuration and normalization for improved performance
- Changed scan topic from `/scan` to `/scan_aligned` in multiple files for consistency.
- Enhanced `scan_frame_normalizer.py` to manage QoS settings for better reliability and reduced latency.
- Updated README and launch files to reflect changes in scan topic and normalization parameters.

File: puzzlebot_description/urdf/puzzlebot.urdf (robot description, URDF)
Before this commit: robot puzzlebot, 6 links, 5 joints
Links:
- removed link caster_link
- removed link wheel_l_link
- removed link wheel_r_link
- added link caster_wheel, mass 0.05; collision sphere radius=0.015; visual mesh filename=package://puzzlebot_description/meshes/Puzzlebot_Caster_Whe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
- added link wheel_left, mass 0.2; collision cylinder length=0.02 radius=0.0325; visual mesh filename=package://puzzlebot_description/meshes/Puzzlebot_Wheel.stl
- added link wheel_right, mass 0.2; collision cylinder length=0.02 radius=0.0325; visual mesh filename=package://puzzlebot_description/meshes/Puzzlebot_Wheel.stl
- link base_footprint: mass None -> 0.001
- link base_link: geometry collision box size=0.20 0.19 0.06; visual mesh filename=package://puzzlebot_description/meshes/Puzzlebot_Jetson_Lid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
Joints:
- removed joint caster_joint
- removed joint wheel_l_joint
- removed joint wheel_r_joint
- added joint caster_wheel_joint: type fixed, parent base_link, child caster_wheel, origin xyz=-0.095 0 -0.03 rpy=0 0 0
- added joint wheel_left_joint: type continuous, parent base_link, child wheel_left, origin xyz=0.052 0.095 -0.0025 rpy=0 0 0, axis 0 1 0
- added joint wheel_right_joint: type continuous, parent base_link, child wheel_right, origin xyz=0.052 -0.095 -0.0025 rpy=0 0 0, axis 0 1 0
- joint base_link_joint: origin xyz=0 0 0.05 -> xyz=-0.052 0 0.05 rpy=0 0 0
- joint laser_joint: origin xyz=0.08 0 0.10 -> xyz=0.00 0 0.15; parent base_link -> base_footprint

Commit message: feat: Refactor SLAM and navigation configurations for improved functionality and performance

File: puzzlebot_description/urdf/puzzlebot.urdf (robot description, URDF)
Before this commit: robot puzzlebot, 6 links, 5 joints
Links:
- link base_link: geometry collision box size=0.20 0.19 0.14; visual mesh filename=package://puzzlebot_description/meshes/Puzzlebot_Jetson_Lid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
- link wheel_left: geometry collision cylinder length=0.02 radius=0.047; visual mesh filename=package://puzzlebot_description/meshes/Puzzlebot_Wheel.stl
- link wheel_right: geometry collision cylinder length=0.02 radius=0.047; visual mesh filename=package://puzzlebot_description/meshes/Puzzlebot_Wheel.stl
Joints:
- joint base_link_joint: origin xyz=-0.052 0 0.05 rpy=0 0 0 -> xyz=0.052 0 0.05 rpy=0 0 0
- joint caster_wheel_joint: origin xyz=-0.095 0 -0.03 rpy=0 0 0 -> xyz=-0.147 0 -0.045 rpy=0 0 0
- joint laser_joint: origin xyz=0.00 0 0.15 -> xyz=0.00 0 0.10; parent base_footprint -> base_link
- joint wheel_left_joint: origin xyz=0.052 0.095 -0.0025 rpy=0 0 0 -> xyz=0.00 0.095 -0.000 rpy=0 0 0
- joint wheel_right_joint: origin xyz=0.052 -0.095 -0.0025 rpy=0 0 0 -> xyz=0.00 -0.095 -0.000 rpy=0 0 0

Commit message: fix: Update collision geometry and adjust initial pose for improved simulation accuracy

File: puzzlebot_description/urdf/puzzlebot.urdf (robot description, URDF)
Before this commit: robot puzzlebot, 6 links, 5 joints
Links:
- link base_link: geometry collision box size=0.2 0.14 0.10; visual mesh filename=package://puzzlebot_description/meshes/Puzzlebot_Jetson_Lid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
- link wheel_left: geometry collision cylinder length=0.02 radius=0.032; visual mesh filename=package://puzzlebot_description/meshes/Puzzlebot_Wheel.stl
- link wheel_right: geometry collision cylinder length=0.02 radius=0.032; visual mesh filename=package://puzzlebot_description/meshes/Puzzlebot_Wheel.stl
