Commit message: Update navigation and SLAM configurations, replace map files, and add RViz configuration
- Updated CMakeLists.txt to include 'maps' directory in installation.
- Changed 'use_sim_time' parameter to true in nav2_params.yaml.
- Updated planner plugin path in nav2_params.yaml.
- Changed map file reference from 'map_maze.yaml' to 'my_maze.yaml' in nav2.launch.xml and nav2_core.launch.xml.
- Added 'launch_rviz' argument to slam.launch.xml and slam_core.launch.xml.
- Updated RViz configuration file to 'nav2.rviz' and added detailed visualization settings.
- Deleted old map files (map_maze.pgm and map_maze.yaml) and added new map files (my_maze.pgm and my_maze.yaml) with updated origin.

Co-authored-by: EmanuelVegaGlz <emanuelvegaglz@users.noreply.github.com>
Co-authored-by: Diego Quezada <diegoquezadaco@users.noreply.github.com>
Co-authored-by: BrisaReyCa <brisa.reyes.castro@outlook.com>

File: puzzlebot_description/urdf/mcr2_control/puzzlebot_control.xacro (robot description, xacro)
@@ -42,22 +42,14 @@
         </plugin>
         <plugin filename="gz-sim-joint-state-publisher-system" name="gz::sim::systems::JointStatePublisher">
-            <topic>${prefix}joint_states</topic>
+            <topic>/${prefix}joint_states</topic>
             <update_rate>50</update_rate>
             <joint_name>${prefix}wheel_right_joint</joint_name>
             <joint_name>${prefix}wheel_left_joint</joint_name>
         </plugin>
-        <plugin
-                filename="gz-sim-sensors-system"
-                name="gz::sim::systems::Sensors">
-                <render_engine>ogre2</render_engine>
-        </plugin>
-        <plugin filename="gz-sim-odometry-publisher-system" name="gz::sim::systems::OdometryPublisher">
-            <odom_frame>world</odom_frame>
-            <robot_base_frame>${prefix}base_footprint</robot_base_frame>
-            <odom_publish_frequency>50</odom_publish_frequency>
-            <odom_topic>${prefix}ground_truth</odom_topic>
-            <tf_topic>tf</tf_topic>
-            <dimensions>2</dimensions>
-        </plugin>
+        <!-- <plugin
+            filename="gz-sim-sensors-system"
+            name="gz::sim::systems::Sensors">
+            <render_engine>ogre2</render_engine>
+        </plugin> -->
     </gazebo>
 </xacro:macro>

File: puzzlebot_description/urdf/mcr2_robots/jetson_lidar_ed/parameters_jetson_lidar_ed.xacro (robot description, xacro)
@@ -32,5 +32,5 @@
             <xacro:property name="chassis_mesh_pos_w" value="0.0"/>
         <!--Chassis Joint parameters-->
-            <xacro:property name="chassis_pos_x" value="0.0"/>
+            <xacro:property name="chassis_pos_x" value="-0.052"/>
             <xacro:property name="chassis_pos_y" value="0.0"/>
             <xacro:property name="chassis_pos_z" value="0.05"/>
@@ -165,7 +165,7 @@
             <xacro:property name="jetson_pos_w" value="0.0"/>
     <!--Meshes -->
-        <xacro:property name="mesh_puzzlebot_chassis"  value="$(find puzzlebot_description)/meshes/bases/Puzzlebot_Jetson_Lidar_Edition_Base.stl" />
-        <xacro:property name="mesh_puzzlebot_wheel"  value="$(find puzzlebot_description)/meshes/wheels/Puzzlebot_Wheel.stl" />
-        <xacro:property name="mesh_puzzlebot_caster"  value="$(find puzzlebot_description)/meshes/wheels/Puzzlebot_Caster_Wheel.stl" />
-        <xacro:property name="mesh_puzzlebot_jetson"  value="$(find puzzlebot_description)/meshes/misc/NVIDIA_Jetson.stl" />
+        <xacro:property name="mesh_puzzlebot_chassis"  value="$(find puzzlebot_description)/meshes/Puzzlebot_Jetson_Lidar_Edition_Base.stl" />
+        <xacro:property name="mesh_puzzlebot_wheel"  value="$(find puzzlebot_description)/meshes/Puzzlebot_Wheel.stl" />
+        <xacro:property name="mesh_puzzlebot_caster"  value="$(find puzzlebot_description)/meshes/Puzzlebot_Caster_Wheel.stl" />
+        <xacro:property name="mesh_puzzlebot_jetson"  value="$(find puzzlebot_description)/meshes/Puzzlebot_Caster_Wheel.stl" />
 </robot>

File: puzzlebot_description/urdf/mcr2_robots/puzzlebot_jetson_lidar_ed.xacro (robot description, xacro)
@@ -9,5 +9,5 @@
 <xacro:include filename="$(find puzzlebot_description)/urdf/mcr2_sensors/laser_camera_bracket.xacro" />
 <xacro:include filename="$(find puzzlebot_description)/urdf/mcr2_sensors/lidar.xacro" />
-<xacro:include filename="$(find puzzlebot_description)/urdf/mcr2_control/gazebo_control.xacro" />
+<xacro:include filename="$(find puzzlebot_description)/urdf/mcr2_control/puzzlebot_control.xacro" />
 <!--LINKS-->
 <xacro:puzzlebot_jetson_lidar_ed_base prefix="$(arg prefix)" />

File: puzzlebot_description/urdf/mcr2_sensors/laser_camera_bracket.xacro (robot description, xacro)
@@ -6,5 +6,5 @@
     camera_name:='cam_1'
     parent:='base_link'
-    mesh_file:='file://$(find puzzlebot_description)/meshes/sensors/Laser_Camera_Bracket.stl'
+    mesh_file:='file://$(find puzzlebot_description)/meshes/Puzzlebot_Caster_Wheel.stl'
     camera_base_mass:='0.035'
     camera_base_length:='0.046'

File: puzzlebot_description/urdf/mcr2_sensors/lidar.xacro (robot description, xacro)
@@ -6,5 +6,5 @@
     frame_name:='laser_frame'
     parent:='base_link'
-    mesh_file:='file://$(find puzzlebot_description)/meshes/sensors/RPLidar.stl'
+    mesh_file:='file://$(find puzzlebot_description)/meshes/Puzzlebot_Caster_Wheel.stl'
     lidar_base_mass:='0.1755'
     lidar_base_length:='0.08'
